Commit message: Cleanup telemetry.

File: data/cart_two_poles/cart_two_poles.urdf (robot description, URDF)
Before this commit: robot physics, 4 links, 3 joints
Links:
- link cart: geometry collision mesh filename=package://cart_two_poles/cart.STL; visual mesh filename=package://cart_two_poles/cart.STL
- link pole1: geometry collision mesh filename=package://cart_two_poles/pole1.STL; visual mesh filename=package://cart_two_poles/pole1.STL
- link pole2: geometry collision mesh filename=package://cart_two_poles/pole2.STL; visual mesh filename=package://cart_two_poles/pole2.STL
- link slideBar: geometry visual mesh filename=package://cart_two_poles/slideBar.STL

File: data/double_cartpole/double_cartpole.urdf (robot description, URDF)
Before this commit: robot physics, 6 links, 5 joints
Links:
- link PendulumArm: geometry visual mesh filename=package://double_cartpole/PendulumArm.STL
- link PendulumMass: geometry visual mesh filename=package://double_cartpole/PendulumMass.STL
- link SecondPendulumArm: geometry visual mesh filename=package://double_cartpole/SecondPendulumArm.STL
- link SecondPendulumMass: geometry visual mesh filename=package://double_cartpole/SecondPendulumMass.STL
- link cart: geometry collision mesh filename=package://double_cartpole/cart.STL; visual mesh filename=package://double_cartpole/cart.STL
- link slideBar: geometry visual mesh filename=package://double_cartpole/slideBar.STL

File: data/double_pendulum/double_pendulum.urdf (robot description, URDF)
Before this commit: robot pendulum, 5 links, 4 joints
Links:
- link PendulumArm: geometry visual mesh filename=package://double_pendulum/SecondPendulumArm.STL
- link PendulumMass: geometry visual mesh filename=package://double_pendulum/SecondPendulumMass.STL
- link SecondPendulumArm: geometry visual mesh filename=package://double_pendulum/PendulumArm.STL
- link SecondPendulumMass: geometry visual mesh filename=package://double_pendulum/PendulumMass.STL
- link world: geometry visual mesh filename=package://double_pendulum/world.STL

File: data/simple_pendulum/simple_pendulum.urdf (robot description, URDF)
Before this commit: robot pendulum, 7 links, 6 joints
Links:
- link Foot: geometry visual mesh filename=package://simple_pendulum/Foot.STL
- link PendulumArm: geometry visual mesh filename=package://simple_pendulum/PendulumArm.STL
- link PendulumMass: geometry visual mesh filename=package://simple_pendulum/PendulumMass.STL
