Commit message: [jiminy_py] Add jupyter notebook tutorial to document basic usage.

File: data/simple_pendulum/simple_pendulum.urdf (robot description, URDF)
Before this commit: robot pendulum, 7 links, 6 joints
Joints:
- joint PendulumJoint: axis 0 1 0 -> 1 0 0; limit lower=-1.5 upper=1.5 effort=1000 velocity=100 -> lower=-100 upper=100 effort=1000 velocity=100

Commit message: Fix simple pendulum example script.

File: data/simple_pendulum/simple_pendulum.urdf (robot description, URDF)
Before this commit: robot pendulum, 7 links, 6 joints
Joints:
- joint Corner1Joint: origin xyz=0.1 0.1 0.0 rpy=0 0 0 -> xyz=0.1 0.1 0.0 rpy=0.0 0.0 0.0
- joint Corner2Joint: origin xyz=0.1 -0.1 0.0 rpy=0 0 0 -> xyz=0.1 -0.1 0.0 rpy=0.0 0.0 0.0
- joint Corner3Joint: origin xyz=-0.1 -0.1 0.0 rpy=0 0 0 -> xyz=-0.1 -0.1 0.0 rpy=0.0 0.0 0.0
- joint Corner4Joint: origin xyz=-0.1 0.1 0.0 rpy=0 0 0 -> xyz=-0.1 0.1 0.0 rpy=0.0 0.0 0.0
- joint PendulumJoint: origin xyz=0.0 0.0 0.0 rpy=0 0 0 -> xyz=0.0 0.0 0.0 rpy=0.0 0.0 0.0
- joint PendulumMassJoint: origin xyz=0.0 0.0 1.0 rpy=0 0 0 -> xyz=0.0 0.0 1.0 rpy=0.0 0.0 0.0
