Commit message: Use packages for mesh import.

File: data/cartpole/cartpole.urdf (robot description, URDF)
Before this commit: robot physics, 3 links, 2 joints
Links:
- link cart: geometry collision mesh filename=package://cartpole/cart.STL; visual mesh filename=package://cartpole/cart.STL
- link pole: geometry collision mesh filename=package://cartpole/pole.STL; visual mesh filename=package://cartpole/pole.STL
- link slideBar: geometry visual mesh filename=package://cartpole/slideBar.STL

Commit message: Refactoring of Gym Jiminy to extract more information from the model instead of using hardcoded values.

File: data/cartpole/cartpole.urdf (robot description, URDF)
Before this commit: robot physics, 3 links, 2 joints
Joints:
- joint cart_to_pole: limit lower=-10 upper=10 effort=1000.0 velocity=1000 -> lower=-10.0 upper=10.0 effort=1000.0 velocity=100.0
- joint slider_to_cart: limit lower=-5 upper=5 effort=1000.0 velocity=1000 -> lower=-5.0 upper=5.0 effort=1000.0 velocity=100.0
