Commit message: [misc] Move meshes in subdirectories.

File: data/toys_models/cart_two_poles/cart_two_poles.urdf (robot description, URDF)
Before this commit: robot physics, 4 links, 3 joints
Links:
- link cart: geometry collision mesh filename=package://meshes/cart_two_poles/cart.STL; visual mesh filename=package://meshes/cart_two_poles/cart.STL
- link pole1: geometry collision mesh filename=package://meshes/cart_two_poles/pole1.STL; visual mesh filename=package://meshes/cart_two_poles/pole1.STL
- link pole2: geometry collision mesh filename=package://meshes/cart_two_poles/pole2.STL; visual mesh filename=package://meshes/cart_two_poles/pole2.STL
- link slideBar: geometry visual mesh filename=package://meshes/cart_two_poles/slideBar.STL

File: data/toys_models/cartpole/cartpole.urdf (robot description, URDF)
Before this commit: robot physics, 3 links, 2 joints
Links:
- link cart: geometry collision mesh filename=package://meshes/cartpole/cart.STL; visual mesh filename=package://meshes/cartpole/cart.STL
- link pole: geometry collision mesh filename=package://meshes/cartpole/pole.STL; visual mesh filename=package://meshes/cartpole/pole.STL
- link slideBar: geometry visual mesh filename=package://meshes/cartpole/slideBar.STL

File: data/toys_models/double_cartpole/double_cartpole.urdf (robot description, URDF)
Before this commit: robot physics, 6 links, 5 joints
Links:
- link PendulumArm: geometry visual mesh filename=package://meshes/double_cartpole/PendulumArm.STL
- link PendulumMass: geometry visual mesh filename=package://meshes/double_cartpole/PendulumMass.STL
- link SecondPendulumArm: geometry visual mesh filename=package://meshes/double_cartpole/SecondPendulumArm.STL
- link SecondPendulumMass: geometry visual mesh filename=package://meshes/double_cartpole/SecondPendulumMass.STL
- link cart: geometry collision mesh filename=package://meshes/double_cartpole/cart.STL; visual mesh filename=package://meshes/double_cartpole/cart.STL
- link slideBar: geometry visual mesh filename=package://meshes/double_cartpole/slideBar.STL

File: data/toys_models/double_pendulum/double_pendulum.urdf (robot description, URDF)
Before this commit: robot pendulum, 5 links, 4 joints
Links:
- link PendulumArm: geometry visual mesh filename=package://meshes/double_pendulum/SecondPendulumArm.STL
- link PendulumMass: geometry visual mesh filename=package://meshes/double_pendulum/SecondPendulumMass.STL
- link SecondPendulumArm: geometry visual mesh filename=package://meshes/double_pendulum/PendulumArm.STL
- link SecondPendulumMass: geometry visual mesh filename=package://meshes/double_pendulum/PendulumMass.STL
- link world: geometry visual mesh filename=package://meshes/double_pendulum/world.STL

File: data/toys_models/simple_pendulum/simple_pendulum.urdf (robot description, URDF)
Before this commit: robot pendulum, 7 links, 6 joints
Links:
- link Foot: geometry visual mesh filename=package://meshes/simple_pendulum/Foot.STL
- link PendulumArm: geometry visual mesh filename=package://meshes/simple_pendulum/PendulumArm.STL
- link PendulumMass: geometry visual mesh filename=package://meshes/simple_pendulum/PendulumMass.STL

Commit message: [python] Remove meshes and use primitives for toys models.

File: data/toys_models/cart_two_poles/cart_two_poles.urdf (robot description, URDF)
Before this commit: robot physics, 4 links, 3 joints
Links:
- link cart: geometry collision box size=0.5 0.5 0.2; visual box size=0.5 0.5 0.2
- link pole1: geometry collision box size=0.05 0.05 1.0; visual box size=0.05 0.05 1.0
- link pole2: geometry collision box size=0.05 0.05 1.6; visual box size=0.05 0.05 1.6
- link slideBar: geometry visual box size=30 0.05 0.05

File: data/toys_models/cartpole/cartpole.urdf (robot description, URDF)
Before this commit: robot physics, 3 links, 2 joints
Links:
- link cart: geometry collision box size=0.5 0.5 0.2; visual box size=0.5 0.5 0.2
- link pole: geometry collision box size=0.05 0.05 1.0; visual box size=0.05 0.05 1.0
- link slideBar: geometry visual box size=30 0.05 0.05

File: data/toys_models/double_cartpole/double_cartpole.urdf (robot description, URDF)
Before this commit: robot physics, 6 links, 5 joints
Links:
- link PendulumArm: geometry visual box size=0.02 0.02 1.0
- link PendulumMass: geometry visual sphere radius=0.06
- link SecondPendulumArm: geometry visual box size=0.01 0.01 0.5
- link SecondPendulumMass: geometry visual sphere radius=0.06
- link cart: geometry collision box size=0.5 0.5 0.2; visual box size=0.5 0.5 0.2
- link slideBar: geometry visual box size=30 0.05 0.05

File: data/toys_models/double_pendulum/double_pendulum.urdf (robot description, URDF)
Before this commit: robot pendulum, 5 links, 4 joints
Links:
- link PendulumArm: geometry visual box size=0.01 0.01 0.5
- link PendulumMass: geometry visual sphere radius=0.06
- link SecondPendulumArm: geometry visual box size=0.02 0.02 1.0
- link SecondPendulumMass: geometry visual sphere radius=0.06
- link world: geometry visual sphere radius=0.005

File: data/toys_models/simple_pendulum/simple_pendulum.urdf (robot description, URDF)
Before this commit: robot pendulum, 7 links, 6 joints
Links:
- link Foot: geometry visual box size=0.2 0.2 0.01
- link PendulumArm: geometry visual box size=0.01 0.01 1.0
- link PendulumMass: geometry visual sphere radius=0.06
