Commit message: [misc] Fix Atlas collision sphere size to fix display in Meshcat.

File: data/bipedal_robots/atlas/atlas_v5.urdf (robot description, URDF)
Before this commit: robot atlas, 70 links, 69 joints
Links:
- link l_foot: geometry collision mesh filename=package://meshes/l_foot_chull.obj; collision sphere radius=0.001
- link r_foot: geometry collision mesh filename=package://meshes/r_foot_chull.obj; collision sphere radius=0.001
