Commit message: [gym/env] Update Atlas learning environment.

File: data/bipedal_robots/atlas/atlas.urdf (robot description, URDF)
Before this commit: robot atlas, 31 links, 30 joints
Links:
- link head: mass 1.41984 -> 1.4199
- link l_hand: mass 1.0 -> 0.5839
- link l_lfarm: mass 2.509 -> 0.648
- link l_ufarm: mass 4.386 -> 2.4798
- link r_hand: mass 1.0 -> 0.5839
- link r_lfarm: mass 2.509 -> 0.648
- link r_ufarm: mass 4.386 -> 2.4798
Joints:
- joint back_bkx: origin xyz=0 0 0.05 rpy=0 -0 0 -> xyz=0 0 0.05 rpy=0 0 0
- joint back_bky: origin xyz=0 0 0.162 rpy=0 -0 0 -> xyz=0 0 0.162 rpy=0 0 0
- joint back_bkz: origin xyz=-0.0125 0 0 rpy=0 -0 0 -> xyz=-0.0125 0 0 rpy=0 0 0
- joint l_arm_elx: origin xyz=0 -0.119 0.0092 rpy=0 -0 0 -> xyz=0 -0.119 0.0092 rpy=0 0 0
- joint l_arm_ely: origin xyz=0 -0.187 -0.016 rpy=0 -0 0 -> xyz=0 -0.187 -0.016 rpy=0 0 0
- joint l_arm_shx: origin xyz=0 -0.11 -0.245 rpy=0 -0 0 -> xyz=0 -0.11 -0.245 rpy=0 0 0
- joint l_arm_wrx: limit lower=-1.1781 upper=1.1781 effort=25 velocity=12 -> lower=-1.7628 upper=1.7628 effort=25 velocity=10
- joint l_arm_wry: limit lower=0 upper=3.14159 effort=25 velocity=12 -> lower=-3.011 upper=3.011 effort=25 velocity=10
- joint l_arm_wry2: axis 0 1 0 -> -0.0 -1.0 -0.0; limit lower=-0.001 upper=0.001 effort=5 velocity=1 -> lower=-2.9671 upper=2.9671 effort=25 velocity=10
- joint l_leg_akx: limit lower=-0.8 upper=0.8 effort=45 velocity=12 -> lower=-0.8 upper=0.8 effort=360 velocity=12; origin xyz=0 0 0 rpy=0 -0 0 -> xyz=0 0 0 rpy=0 0 0
- joint l_leg_aky: limit lower=-1 upper=0.7 effort=92 velocity=12 -> lower=-1 upper=0.7 effort=740 velocity=12; origin xyz=0 0 -0.422 rpy=0 -0 0 -> xyz=0 0 -0.422 rpy=0 0 0
- joint l_leg_hpx: origin xyz=0 0 0 rpy=0 -0 0 -> xyz=0 0 0 rpy=0 0 0
- joint l_leg_hpy: origin xyz=0.05 0.0225 -0.066 rpy=0 -0 0 -> xyz=0.05 0.0225 -0.066 rpy=0 0 0
- joint l_leg_hpz: origin xyz=0 0.089 0 rpy=0 -0 0 -> xyz=0 0.089 0 rpy=0 0 0
- joint l_leg_kny: origin xyz=-0.05 0 -0.374 rpy=0 -0 0 -> xyz=-0.05 0 -0.374 rpy=0 0 0
- joint neck_ry: limit lower=-0.602139 upper=1.14319 effort=5 velocity=6.28 -> lower=-0.602139 upper=1.14319 effort=25 velocity=6.28; origin xyz=0.2546 0 0.6215 rpy=0 -0 0 -> xyz=0.2546 0 0.6215 rpy=0 0 0
- joint r_arm_elx: origin xyz=0 -0.119 0.0092 rpy=0 -0 0 -> xyz=0 -0.119 0.0092 rpy=0 0 0
- joint r_arm_ely: origin xyz=0 -0.187 -0.016 rpy=0 -0 0 -> xyz=0 -0.187 -0.016 rpy=0 0 0
- joint r_arm_shx: origin xyz=0 -0.11 -0.245 rpy=0 -0 0 -> xyz=0 -0.11 -0.245 rpy=0 0 0
- joint r_arm_shz: origin xyz=0.1406 -0.2256 0.4776 rpy=0 -0 0 -> xyz=0.1406 -0.2256 0.4776 rpy=0 0 0
- joint r_arm_wrx: limit lower=-1.1781 upper=1.1781 effort=25 velocity=12 -> lower=-1.7628 upper=1.7628 effort=25 velocity=10; origin xyz=0 -0.119 0.0092 rpy=0 -0 0 -> xyz=0 -0.119 0.0092 rpy=0 0 0
- joint r_arm_wry: limit lower=0 upper=3.14159 effort=25 velocity=12 -> lower=-3.011 upper=3.011 effort=25 velocity=10; origin xyz=0 -0.187 -0.0092 rpy=0 -0 0 -> xyz=0 -0.187 -0.0092 rpy=0 0 0
- joint r_arm_wry2: limit lower=-0.001 upper=0.001 effort=5 velocity=1 -> lower=-2.9671 upper=2.9671 effort=25 velocity=10
- joint r_leg_akx: limit lower=-0.8 upper=0.8 effort=45 velocity=12 -> lower=-0.8 upper=0.8 effort=360 velocity=12; origin xyz=0 0 0 rpy=0 -0 0 -> xyz=0 0 0 rpy=0 0 0
- joint r_leg_aky: limit lower=-1 upper=0.7 effort=92 velocity=12 -> lower=-1 upper=0.7 effort=740 velocity=12; origin xyz=0 0 -0.422 rpy=0 -0 0 -> xyz=0 0 -0.422 rpy=0 0 0
- joint r_leg_hpx: origin xyz=0 0 0 rpy=0 -0 0 -> xyz=0 0 0 rpy=0 0 0
- joint r_leg_hpy: origin xyz=0.05 -0.0225 -0.066 rpy=0 -0 0 -> xyz=0.05 -0.0225 -0.066 rpy=0 0 0
- joint r_leg_hpz: origin xyz=0 -0.089 0 rpy=0 -0 0 -> xyz=0 -0.089 0 rpy=0 0 0
- joint r_leg_kny: origin xyz=-0.05 0 -0.374 rpy=0 -0 0 -> xyz=-0.05 0 -0.374 rpy=0 0 0
