Commit message: [gym] Improve robustness of learning unit tests.

File: data/toys_models/acrobot/acrobot.urdf (robot description, URDF)
Before this commit: robot acrobot, 4 links, 3 joints
Joints:
- joint FirstArmJoint: limit effort=1.0 velocity=12.566 -> effort=1000.0 velocity=12.566

Commit message: [core] Various minor improvements.

File: data/toys_models/acrobot/acrobot.urdf (robot description, URDF)
Before this commit: robot acrobot, 4 links, 3 joints
Links:
- link FirstArm: geometry visual box size=0.04 0.04 1.0; visual sphere radius=0.05
- link world: mass 0.0 -> None; geometry 

File: unit_py/data/box_collision_mesh.urdf (robot description, URDF)
Before this commit: robot box, 2 links, 1 joints
Links:
- removed link root
Joints:
- removed joint base

File: unit_py/data/point_mass.urdf (robot description, URDF)
Before this commit: robot point_mass, 2 links, 1 joints
Links:
- removed link root
Joints:
- removed joint base

File: unit_py/data/sphere_primitive.urdf (robot description, URDF)
Before this commit: robot sphere, 2 links, 1 joints
Links:
- removed link root
Joints:
- removed joint base
