Commit message: [core] Log the acceleration both at the end and the beginning of a step if dynamics has changed.

File: python/jiminy_py/unit_py/data/double_pendulum.urdf (robot description, URDF)
Before this commit: robot pendulum, 5 links, 4 joints
Links:
- link PendulumMass: mass 3.0 -> 10.0
- link SecondPendulumMass: mass 2.0 -> 10.0
Joints:
- joint PendulumJoint: axis 1 0 0 -> 0 1 0
- joint SecondPendulumJoint: axis 1 0 0 -> 0 1 0
