Commit message: [gym] Refactor Acrobot and Cartpole RL envs in accordance to official OpenAI Gym implementations.

File: data/toys_models/cartpole/cartpole.urdf (robot description, URDF)
Before this commit: robot physics, 3 links, 2 joints
Links:
- link cart: mass 1 -> 1.0; geometry visual box size=0.5 0.5 0.2
- link pole: mass 10 -> 0.1; geometry visual box size=0.05 0.05 1.0
- link slideBar: mass 0 -> 0.0
Joints:
- joint cart_to_pole: limit lower=-10.0 upper=10.0 effort=1000.0 velocity=100.0 -> lower=-6.2832 upper=6.2832 effort=1000.0 velocity=100.0; origin xyz=0.0 0.0 0.0 rpy=0 0 0 -> xyz=0.0 0.0 0.0 rpy=0.0 0.0 0.0
- joint slider_to_cart: limit lower=-5.0 upper=5.0 effort=1000.0 velocity=100.0 -> lower=-10.0 upper=10.0 effort=10.0 velocity=100.0; origin xyz=0.0 0.0 0.0 -> xyz=0.0 0.0 0.0 rpy=0.0 0.0 0.0

Commit message: [misc] Add mass fixed frame with visual to cartpole.

File: data/toys_models/cartpole/cartpole.urdf (robot description, URDF)
Before this commit: robot cartpole, 3 links, 2 joints
Links:
- added link mass; visual sphere radius=0.05
Joints:
- added joint pole_to_mass: type fixed, parent pole, child mass, origin xyz=0.0 0.0 1.0 rpy=0.0 0.0 0.0

Commit message: [core] Attach encoders on motors or joints. Define position limits at motor level.

File: data/toys_models/cartpole/cartpole.urdf (robot description, URDF)
Before this commit: robot cartpole, 4 links, 3 joints
Joints:
- joint cart_to_pole: limit lower=-6.2832 upper=6.2832 effort=1000.0 velocity=100.0 -> effort=1000.0 velocity=100.0; type revolute -> continuous
